File: Solar-Buck-Boost.kicad_sch (KiCad schematic)
At the start: 29 parts, among them CN1 2001SMT-2P_C132500, J1 Conn_01x02_Pin, J2 Conn_01x01_Pin, J3 Conn_01x01_Pin, Q1 AO3401A_C347476, U1 CN3063, U3 TPS63020DSJR

Commit message: Schematics fix
Other:
- note added: "1.02"
- note added: "Developed By: Juan Flores Muñoz (jfm92)"
- note added: "Solar Buck Boost"
- moved on the sheet: J2, J3, R7, R8
